File: motors.kicad_sch (KiCad schematic)
At the start: 4 parts

Commit message: idek
Parts:
- U3, U4, U5, U6: renamed from U?; footprint (none) -> esc:esc
Connections:
- net GND: now reaches U4.2 (-V_in)
- net GND: now also U3.2 (-V_in), U5.2 (-V_in), U6.2 (-V_in)
Changed lines of the file:
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@@
 	(generator_version "9.0")
 	(paper "A4")
+	(hierarchical_label "GND"
+		(shape input)
+		(at 40.64 63.5 0)
+		(effects
+			(font
+				(size 1.27 1.27)
+			)
+			(justify left)
+		)
+	)
+	(hierarchical_label "GND"
+		(shape input)
+		(at 40.64 49.53 0)
+		(effects
+			(font
+				(size 1.27 1.27)
+			)
+			(justify left)
+		)
+	)
 	(hierarchical_label "+V"
 		(shape input)
@@
 		(shape input)
 		(at 40.64 46.99 0)
+		(effects
+			(font
+				(size 1.27 1.27)
+			)
+			(justify left)
+		)
+	)
+	(hierarchical_label "GND"
+		(shape input)
+		(at 40.64 77.47 0)
+		(effects
+			(font
+				(size 1.27 1.27)
+			)
+			(justify left)
+		)
+	)
+	(hierarchical_label "GND"
+		(shape input)
+		(at 40.64 36.83 0)
 		(effects
 			(font
@@
 		(on_board yes)
 		(dnp no)
-		(property "Reference" "U?"
+		(property "Reference" "U4"
 			(at 35.56 41.91 0)
 			(effects
@@
 			)
 		)
-		(property "Footprint" ""
+		(property "Footprint" "esc:esc"
 			(at 35.56 50.8 0)
 			(effects
@@
 			(project "auv_pcb"
 				(path "/e8907c08-8650-4764-8307-d7b0333da0bd/c75bd509-78bf-411c-83b5-a0a70668dca0"
-					(reference "U?")
+					(reference "U4")
 					(unit 1)
 				)
@@
 		(on_board yes)
 		(dnp no)
-		(property "Reference" "U?"
+		(property "Reference" "U3"
 			(at 35.56 29.21 0)
 			(effects
@@
 			)
 		)
-		(property "Footprint" ""
+		(property "Footprint" "esc:esc"
 			(at 35.56 38.1 0)
 			(effects
@@
 			(project ""
 				(path "/e8907c08-8650-4764-8307-d7b0333da0bd/c75bd509-78bf-411c-83b5-a0a70668dca0"
-					(reference "U?")
+					(reference "U3")
 					(unit 1)
 				)
@@
 		(on_board yes)
 		(dnp no)
-		(property "Reference" "U?"
+		(property "Reference" "U5"
 			(at 35.56 55.88 0)
 			(effects
@@
 			)
 		)
-		(property "Footprint" ""
+		(property "Footprint" "esc:esc"
 			(at 35.56 64.77 0)
 			(effects
@@
 			(project "auv_pcb"
 				(path "/e8907c08-8650-4764-8307-d7b0333da0bd/c75bd509-78bf-411c-83b5-a0a70668dca0"
-					(reference "U?")
+					(reference "U5")
 					(unit 1)
 				)
@@
 		(on_board yes)
 		(dnp no)
-		(property "Reference" "U?"
+		(property "Reference" "U6"
 			(at 35.56 69.85 0)
 			(effects
@@
 			)
 		)
-		(property "Footprint" ""
+		(property "Footprint" "esc:esc"
 			(at 35.56 78.74 0)
 			(effects
@@
 			(project "auv_pcb"
 				(path "/e8907c08-8650-4764-8307-d7b0333da0bd/c75bd509-78bf-411c-83b5-a0a70668dca0"
-					(reference "U?")
+					(reference "U6")
 					(unit 1)
 				)
